Commit message: Update arm controller and arm node for tickle pipeline. Change urdf joint limits

File: src/tickle_taesan_moveit/urdf/astra_dual_so_arm.urdf (robot description, URDF)
Before this commit: robot astra_dual_so_arm, 15 links, 14 joints
Joints:
- joint joint_l2: limit lower=-2.0 upper=2.0 effort=100 velocity=1 -> lower=-1.57 upper=1.57 effort=100 velocity=1
- joint joint_l3: limit lower=-1.75 upper=1.75 effort=100 velocity=1 -> lower=-1.57 upper=1.57 effort=100 velocity=1
- joint joint_l4: limit lower=-1.75 upper=1.57 effort=100 velocity=1 -> lower=-1.57 upper=1.57 effort=100 velocity=1
- joint joint_l5: limit lower=-3.5 upper=0.2 effort=100 velocity=1 -> lower=-1.57 upper=1.57 effort=100 velocity=1
- joint joint_l6: limit lower=-1.0 upper=4.0 effort=100 velocity=1 -> lower=-3.14 upper=3.14 effort=100 velocity=1
- joint joint_l7l: limit lower=-0.22 upper=2.0 effort=100 velocity=1 -> lower=-1.57 upper=1.57 effort=100 velocity=1
- joint joint_r2: limit lower=-2.0 upper=2.0 effort=100 velocity=1 -> lower=-1.57 upper=1.57 effort=100 velocity=1
- joint joint_r3: limit lower=-1.75 upper=1.75 effort=100 velocity=1 -> lower=-1.57 upper=1.57 effort=100 velocity=1
- joint joint_r4: limit lower=-1.75 upper=1.57 effort=100 velocity=1 -> lower=-1.57 upper=1.57 effort=100 velocity=1
- joint joint_r5: limit lower=-3.5 upper=0.2 effort=100 velocity=1 -> lower=-1.57 upper=1.57 effort=100 velocity=1
- joint joint_r6: limit lower=-1.0 upper=4.0 effort=100 velocity=1 -> lower=-3.14 upper=3.14 effort=100 velocity=1
- joint joint_r7r: limit lower=-0.22 upper=2.0 effort=100 velocity=1 -> lower=-1.57 upper=1.57 effort=100 velocity=1
