Commit message: Change joint limits properly

File: src/astra_description/urdf/astra_description.urdf (robot description, URDF)
Before this commit: robot astra_description, 23 links, 22 joints
Joints:
- joint joint_l2: limit lower=-1.57 upper=1.57 effort=35 velocity=1 -> lower=-2 upper=2 effort=35 velocity=1
- joint joint_l3: limit lower=-1.57 upper=1.57 effort=35 velocity=1 -> lower=0 upper=3.5 effort=35 velocity=1
- joint joint_l4: limit lower=-1.57 upper=1.57 effort=35 velocity=1 -> lower=-3.14158 upper=0 effort=35 velocity=1
- joint joint_l5: limit lower=-1.57 upper=1.57 effort=35 velocity=1 -> lower=-2.5 upper=1.2 effort=35 velocity=1
- joint joint_l7l: limit lower=0 upper=1.57 effort=35 velocity=1 -> lower=-0.2 upper=2.0 effort=35 velocity=1
- joint joint_r2: limit lower=-1.57 upper=1.57 effort=35 velocity=1 -> lower=-2 upper=2 effort=35 velocity=1
- joint joint_r3: limit lower=-1.57 upper=1.57 effort=35 velocity=1 -> lower=0 upper=3.5 effort=35 velocity=1
- joint joint_r4: limit lower=-1.57 upper=1.57 effort=35 velocity=1 -> lower=-3.14158 upper=0 effort=35 velocity=1
- joint joint_r5: limit lower=-1.57 upper=1.57 effort=35 velocity=1 -> lower=-2.5 upper=1.2 effort=35 velocity=1
- joint joint_r7r: limit lower=0 upper=1.57 effort=35 velocity=1 -> lower=-0.2 upper=2.0 effort=35 velocity=1

Commit message: fix urdf error

File: src/astra_description/urdf/astra_description.urdf (robot description, URDF)
Before this commit: robot astra_description, 23 links, 22 joints
Joints:
- joint joint_ree_teleop: origin xyz=0.020 0.0 0.200 rpy=0 -1.5708 0 -> xyz=0.020 0.0 0.195 rpy=0 -1.5708 0

Commit message: update left arm moveit configurations symmetric to right arm

File: src/astra_description/urdf/astra_description.urdf (robot description, URDF)
Before this commit: robot astra_description, 23 links, 22 joints
Joints:
- joint joint_lee: axis 0 0 0 -> (none)
- joint joint_lee_teleop: axis 0 0 0 -> (none)

File: src/astra_description/urdf/astra_description_rel.urdf (robot description, URDF)
Before this commit: robot astra_description, 23 links, 22 joints
Joints:
- joint joint_lee: axis 0 0 0 -> (none)
- joint joint_lee_teleop: axis 0 0 0 -> (none)
